File: pcb/gps-tracker.kicad_sch (KiCad schematic)
At the start: 6 parts, among them J1 Conn_Coaxial

Commit message: test
Connections:
- net GND: now reaches C1.2, C2.2, D1.1 (A1), J1.2 (Ext), U1.57 (GND), U1.58 (GND), U1.60 (GND)
- net GND: now also U1.1 (GND), U1.10 (GND), U1.14 (GND), U1.2 (GND), U1.37 (GND), U1.40 (GND), U1.41 (GND), U1.43 (GND), U1.5 (GND), U1.65 (GND), U1.77 (GND), U1.78 (GND), U1.80 (GND), U1.81 (GND)
Changed lines of the file:
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@@
 (kicad_sch (version 20230121) (generator eeschema)
   (paper "A4")
+  (junction (at 132.08 49.53) (diameter 0) (color 0 0 0 0)
+  )
+  (junction (at 132.08 41.91) (diameter 0) (color 0 0 0 0)
+  )
+  (junction (at 132.08 39.37) (diameter 0) (color 0 0 0 0)
+  )
   (junction (at 72.39 41.91) (diameter 0) (color 0 0 0 0)
   )
+  (junction (at 54.61 151.13) (diameter 0) (color 0 0 0 0)
+  )
   (junction (at 26.67 31.75) (diameter 0) (color 0 0 0 0)
   )
+  (junction (at 54.61 158.75) (diameter 0) (color 0 0 0 0)
+  )
   (junction (at 63.5 41.91) (diameter 0) (color 0 0 0 0)
   )
+  (junction (at 54.61 140.97) (diameter 0) (color 0 0 0 0)
+  )
   (junction (at 26.67 41.91) (diameter 0) (color 0 0 0 0)
   )
+  (junction (at 20.32 41.91) (diameter 0) (color 0 0 0 0)
+  )
+  (junction (at 54.61 156.21) (diameter 0) (color 0 0 0 0)
+  )
+  (junction (at 54.61 148.59) (diameter 0) (color 0 0 0 0)
+  )
+  (junction (at 54.61 146.05) (diameter 0) (color 0 0 0 0)
+  )
   (junction (at 50.8 31.75) (diameter 0) (color 0 0 0 0)
   )
@@
   (junction (at 72.39 39.37) (diameter 0) (color 0 0 0 0)
   )
+  (junction (at 54.61 143.51) (diameter 0) (color 0 0 0 0)
+  )
+  (junction (at 54.61 153.67) (diameter 0) (color 0 0 0 0)
+  )
+  (junction (at 54.61 161.29) (diameter 0) (color 0 0 0 0)
+  )
   (junction (at 50.8 41.91) (diameter 0) (color 0 0 0 0)
   )
+  (wire (pts (xy 124.46 39.37) (xy 132.08 39.37))
+    (stroke (width 0) (type default))
+  )
   (wire (pts (xy 26.67 31.75) (xy 50.8 31.75))
     (stroke (width 0) (type default))
   )
+  (wire (pts (xy 132.08 36.83) (xy 132.08 39.37))
+    (stroke (width 0) (type default))
+  )
   (wire (pts (xy 50.8 31.75) (xy 50.8 34.29))
     (stroke (width 0) (type default))
   )
+  (wire (pts (xy 54.61 161.29) (xy 73.66 161.29))
+    (stroke (width 0) (type default))
+  )
   (wire (pts (xy 73.66 36.83) (xy 72.39 36.83))
     (stroke (width 0) (type default))
   )
+  (wire (pts (xy 54.61 153.67) (xy 54.61 151.13))
+    (stroke (width 0) (type default))
+  )
+  (wire (pts (xy 132.08 39.37) (xy 132.08 41.91))
+    (stroke (width 0) (type default))
+  )
+  (wire (pts (xy 20.32 41.91) (xy 20.32 44.45))
+    (stroke (width 0) (type default))
+  )
+  (wire (pts (xy 132.08 52.07) (xy 132.08 49.53))
+    (stroke (width 0) (type default))
+  )
+  (wire (pts (xy 54.61 146.05) (xy 73.66 146.05))
+    (stroke (width 0) (type default))
+  )
+  (wire (pts (xy 54.61 161.29) (xy 54.61 158.75))
+    (stroke (width 0) (type default))
+  )
   (wire (pts (xy 20.32 36.83) (xy 20.32 41.91))
     (stroke (width 0) (type default))
   )
+  (wire (pts (xy 54.61 143.51) (xy 54.61 140.97))
+    (stroke (width 0) (type default))
+  )
+  (wire (pts (xy 54.61 158.75) (xy 73.66 158.75))
+    (stroke (width 0) (type default))
+  )
+  (wire (pts (xy 54.61 158.75) (xy 54.61 156.21))
+    (stroke (width 0) (type default))
+  )
+  (wire (pts (xy 54.61 156.21) (xy 54.61 153.67))
+    (stroke (width 0) (type default))
+  )
+  (wire (pts (xy 54.61 151.13) (xy 73.66 151.13))
+    (stroke (width 0) (type default))
+  )
   (wire (pts (xy 25.4 31.75) (xy 26.67 31.75))
     (stroke (width 0) (type default))
   )
+  (wire (pts (xy 54.61 140.97) (xy 73.66 140.97))
+    (stroke (width 0) (type default))
+  )
   (wire (pts (xy 72.39 36.83) (xy 72.39 39.37))
     (stroke (width 0) (type default))
   )
+  (wire (pts (xy 124.46 36.83) (xy 132.08 36.83))
+    (stroke (width 0) (type default))
+  )
+  (wire (pts (xy 54.61 153.67) (xy 73.66 153.67))
+    (stroke (width 0) (type default))
+  )
   (wire (pts (xy 26.67 40.64) (xy 26.67 41.91))
     (stroke (width 0) (type default))
   )
+  (wire (pts (xy 54.61 156.21) (xy 73.66 156.21))
+    (stroke (width 0) (type default))
+  )
   (wire (pts (xy 50.8 41.91) (xy 63.5 41.91))
     (stroke (width 0) (type default))
@@
     (stroke (width 0) (type default))
   )
+  (wire (pts (xy 54.61 162.56) (xy 54.61 161.29))
+    (stroke (width 0) (type default))
+  )
+  (wire (pts (xy 54.61 148.59) (xy 54.61 146.05))
+    (stroke (width 0) (type default))
+  )
   (wire (pts (xy 72.39 39.37) (xy 72.39 41.91))
     (stroke (width 0) (type default))
@@
     (stroke (width 0) (type default))
   )
+  (wire (pts (xy 54.61 151.13) (xy 54.61 148.59))
+    (stroke (width 0) (type default))
+  )
   (wire (pts (xy 63.5 41.91) (xy 72.39 41.91))
     (stroke (width 0) (type default))
   )
+  (wire (pts (xy 124.46 41.91) (xy 132.08 41.91))
+    (stroke (width 0) (type default))
+  )
+  (wire (pts (xy 132.08 41.91) (xy 132.08 49.53))
+    (stroke (width 0) (type default))
+  )
   (wire (pts (xy 73.66 39.37) (xy 72.39 39.37))
     (stroke (width 0) (type default))
   )
+  (wire (pts (xy 132.08 49.53) (xy 124.46 49.53))
+    (stroke (width 0) (type default))
+  )
+  (wire (pts (xy 54.61 146.05) (xy 54.61 143.51))
+    (stroke (width 0) (type default))
+  )
+  (wire (pts (xy 54.61 143.51) (xy 73.66 143.51))
+    (stroke (width 0) (type default))
+  )
   (wire (pts (xy 20.32 41.91) (xy 26.67 41.91))
     (stroke (width 0) (type default))
   )
+  (wire (pts (xy 54.61 148.59) (xy 73.66 148.59))
+    (stroke (width 0) (type default))
+  )
   (wire (pts (xy 50.8 39.37) (xy 50.8 41.91))
     (stroke (width 0) (type default))
@@
     (stroke (width 0) (type default))
   )
+  (wire (pts (xy 54.61 140.97) (xy 54.61 138.43))
+    (stroke (width 0) (type default))
+  )
   (wire (pts (xy 26.67 41.91) (xy 50.8 41.91))
     (stroke (width 0) (type default))
@@
   (wire (pts (xy 63.5 39.37) (xy 63.5 41.91))
     (stroke (width 0) (type default))
+  )
+  (wire (pts (xy 54.61 138.43) (xy 73.66 138.43))
+    (stroke (width 0) (type default))
+  )
+  (symbol (lib_id "power:GND") (at 54.61 162.56 0) (unit 1)
+    (in_bom yes) (on_board yes) (dnp no)
+    (property "Reference" "#PWR02" (at 54.61 168.91 0)
+      (effects (font (size 1.27 1.27)) hide)
+    )
+    (property "Value" "GND" (at 54.61 166.37 0)
+      (effects (font (size 1.27 1.27)))
+    )
+    (property "Footprint" "" (at 54.61 162.56 0)
+      (effects (font (size 1.27 1.27)) hide)
+    )
+    (property "Datasheet" "" (at 54.61 162.56 0)
+      (effects (font (size 1.27 1.27)) hide)
+    )
+    (pin "1")
+    (instances
+      (project "gps-tracker"
+        (path "/aa2a7d02-83ff-4a9a-93ed-23ca528622b2"
+          (reference "#PWR02") (unit 1)
+        )
+      )
+    )
   )
   (symbol (lib_id "Device:C_Small") (at 50.8 36.83 0) (unit 1)
@@
         )
       )
+    )
+  )
+  (symbol (lib_id "power:GND") (at 132.08 52.07 0) (unit 1)
+    (in_bom yes) (on_board yes) (dnp no)
+    (property "Reference" "#PWR03" (at 132.08 58.42 0)
+      (effects (font (size 1.27 1.27)) hide)
+    )
+    (property "Value" "GND" (at 132.08 55.88 0)
+      (effects (font (size 1.27 1.27)))
+    )
+    (property "Footprint" "" (at 132.08 52.07 0)
+      (effects (font (size 1.27 1.27)) hide)
+    )
+    (property "Datasheet" "" (at 132.08 52.07 0)
+      (effects (font (size 1.27 1.27)) hide)
+    )
+    (pin "1")
+    (instances
+      (project "gps-tracker"
+        (path "/aa2a7d02-83ff-4a9a-93ed-23ca528622b2"
+          (reference "#PWR03") (unit 1)
+        )
+      )
+    )
+  )
+  (symbol (lib_id "power:GND") (at 20.32 44.45 0) (unit 1)
+    (in_bom yes) (on_board yes) (dnp no)
+    (property "Reference" "#PWR01" (at 20.32 50.8 0)
+      (effects (font (size 1.27 1.27)) hide)
+    )
+    (property "Value" "GND" (at 20.32 48.26 0)
+      (effects (font (size 1.27 1.27)))
+    )
+    (property "Footprint" "" (at 20.32 44.45 0)
+      (effects (font (size 1.27 1.27)) hide)
+    )
+    (property "Datasheet" "" (at 20.32 44.45 0)
+      (effects (font (size 1.27 1.27)) hide)
+    )
+    (pin "1")
+    (instances
+      (project "gps-tracker"
+        (path "/aa2a7d02-83ff-4a9a-93ed-23ca528622b2"
+          (reference "#PWR01") (unit 1)
+        )
+      )
