File: pcb/gps-tracker.kicad_pcb (KiCad board)
At the start: 2 copper layers, 6 parts, among them J1 Conn_Coaxial

Commit message: test
Other:
- board outline added: 59.4 x 47.2 mm
Changed lines of the file:
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@@
     )
   )
+  (gr_line (start 167.132 104.14) (end 167.132 72.136)
+    (stroke (width 0.1) (type default)) (layer "Edge.Cuts"))
+  (gr_line (start 108.712 104.648) (end 168.148 105.156)
+    (stroke (width 0.1) (type default)) (layer "Edge.Cuts"))
+  (gr_line (start 168.148 105.156) (end 167.132 104.14)
+    (stroke (width 0.1) (type default)) (layer "Edge.Cuts"))
+  (gr_line (start 167.132 72.136) (end 167.132 57.912)
+    (stroke (width 0.1) (type default)) (layer "Edge.Cuts"))
+  (gr_line (start 167.132 57.912) (end 108.712 57.912)
+    (stroke (width 0.1) (type default)) (layer "Edge.Cuts"))
+  (gr_line (start 108.712 57.912) (end 108.712 104.648)
+    (stroke (width 0.1) (type default)) (layer "Edge.Cuts"))
   (segment (start 126.492 68.072) (end 126.492 67.752001) (width 0.25) (layer "F.Cu") (net 1))
   (segment (start 116.289 59.987) (end 116.289 61.976) (width 0.25) (layer "F.Cu") (net 1))
